File: Pre-Aligner.kicad_pcb (KiCad board)
At the start: 4 copper layers, 230 x 130 mm, 200 parts, among them IC1 THVD1450DGKR, IC2 THVD1450DGKR, IC3 THVD1450DGKR, IC4 THVD1450DGKR, IC5 THVD1450DGKR, IC6 THVD1450DGKR, J1 Conn_02x07_Odd_Even, J10 2355181-4, J13 694108402002, J15 Screw_Terminal_01x02, J2 Micro_SD_Card, J3 Conn_01x04_Male, J4 Conn_01x04_Male, J5 5787834-1, J6 DB9_Male, J7 DB15_Female, J8 2355181-4, J9 2355181-4, Q1 Si2319CDS, Q2 Si2319CDS, SW1 SPST, SW2 SPST, SW5 SPST, U10 MPXA6115A, U11 LMR33630CDDA, U12 TPS54240DGQR, U13 MAX3232, U14 DRV8825_STEPPER_MOTOR_DRIVER_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, U16 UA9637, U19 DRV8825_STEPPER_MOTOR_DRIVER_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, U2 LM1117-3.3, U20 DRV8825_STEPPER_MOTOR_DRIVER_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, U21 OPA340NA, U24 ISO7320C, U3 STM32F407ZET6, U4 TCMD1000, U5 TCMT1600, U6 TPS55340RTER, U7 TCMT1600, U8 TCMD1000, U9 TCMT1600, Y1 8MHZ, Y2 32.768kHz

Commit message: Add files via upload
Parts:
- removed the C24 at (156.1, 139.7)
- removed the C42 at (97.7, 155.9)
- removed the C44 at (87.6, 144.6)
- removed the C46 at (84.7, 144.8)
- removed the C47 at (90.6, 146.0)
- removed the C48 at (107.1, 152.2)
- removed the C50 at (106.6, 153.8)
- removed the C69 at (89.6, 170.9)
- removed the C70 at (92.8, 173.7)
- removed the C73 at (91.8, 175.9)
- removed the C87 at (146.1, 145.7)
- removed the D10 at (103.3, 149.9)
- removed the D11 at (100.9, 161.6)
- removed the J10 at (145.3, 143.8)
- removed J15: Screw_Terminal_01x02, TerminalBlock_TE-Connectivity:TerminalBlock_TE_282834-2_1x02_P2.54mm_Horizontal
- removed the J4 at (173.1, 123.0)
- removed the L3 at (112.4, 153.3)
- removed the R21 at (95.5, 169.9)
- removed the R22 at (91.8, 173.7)
- removed the R23 at (98.0, 166.3)
- removed the R29 at (155.3, 137.1)
- removed the R51 at (145.3, 139.7)
- removed RFB1: 187 kΩ, Resistor_SMD:R_0603_1608Metric
- removed SW5: SPST, Button_Switch_SMD:SW_SPST_TL3342
- removed the U11 at (86.1, 149.2)
- removed the U12 at (102.0, 154.1)
- removed the U3 at (161.9, 107.0)
- removed the U9 at (150.6, 139.6)
- added BZ1: Buzzer, Buzzer_Beeper:MagneticBuzzer_PUI_AT-0927-TT-6-R, F.Cu at (228.9, 104.0)
- added C13: 0.1UF, Capacitor_SMD:C_0603_1608Metric, B.Cu at (126.5, 105.3)
- added C14: 0.1µF, Capacitor_SMD:C_0402_1005Metric, F.Cu at (119.9, 99.8)
- added C15: 0.1µF, Capacitor_SMD:C_0603_1608Metric, B.Cu at (134.1, 100.3)
- added C16: 10µF, Capacitor_SMD:C_1210_3225Metric, F.Cu at (128.6, 88.8)
- added C17: 0.1UF, Capacitor_SMD:C_0603_1608Metric, B.Cu at (130.0, 95.9)
- added C18: 0.1UF, Capacitor_SMD:C_0603_1608Metric, F.Cu at (129.2, 86.1)
- added C19: 0.1UF, Capacitor_SMD:C_0603_1608Metric, F.Cu at (129.2, 83.6)
- added C20: 0.1UF, Capacitor_SMD:C_0603_1608Metric, B.Cu at (126.6, 100.3)
- added C21: 0.1µF, Capacitor_SMD:C_0603_1608Metric, B.Cu at (126.1, 92.9)
- added C29: 0.1UF, Capacitor_SMD:C_0603_1608Metric, B.Cu at (160.2, 115.7)
- added C30: 0.1UF, Capacitor_SMD:C_0603_1608Metric, B.Cu at (134.0, 95.4)
- added C31: 0.1UF, Capacitor_SMD:C_0603_1608Metric, B.Cu at (169.3, 104.7)
- added C52: 0.1µF, Capacitor_SMD:C_0402_1005Metric, B.Cu at (133.5, 108.0)
- added C53: 0.1µF, Capacitor_SMD:C_0402_1005Metric, F.Cu at (154.1, 146.4)
- added C59: 0.1UF, Capacitor_SMD:C_0603_1608Metric, B.Cu at (144.6, 157.2)
- added C61: 0.1µF, Capacitor_SMD:C_0402_1005Metric, B.Cu at (148.7, 161.2)
- added C75: 22nF, Capacitor_SMD:C_0603_1608Metric, F.Cu at (85.5, 172.9)
- added C76: 0.1µF, Capacitor_SMD:C_0603_1608Metric, F.Cu at (98.1, 156.8)
- added C77: 1nF, Capacitor_SMD:C_0603_1608Metric, F.Cu at (85.9, 175.4)
- added C78: 47nF, Capacitor_SMD:C_0603_1608Metric, F.Cu at (85.1, 177.8)
- added C8: 0.1UF, Capacitor_SMD:C_0603_1608Metric, F.Cu at (253.7, 88.0)
- added C81: 1µF, Capacitor_SMD:C_0603_1608Metric, B.Cu at (98.7, 130.4)
- added C82: 100µF 50V, Capacitor_SMD:CP_Elec_10x10, F.Cu at (124.3, 159.0)
- added C85: 0.1µF, Capacitor_SMD:C_0402_1005Metric, F.Cu at (133.7, 167.3)
- added C88: 10uF, Capacitor_SMD:C_0603_1608Metric, F.Cu at (106.8, 130.4)
- added C9: 0.1UF, Capacitor_SMD:C_0603_1608Metric, F.Cu at (270.1, 91.9)
- added C90: 10uF, Capacitor_SMD:C_0603_1608Metric, F.Cu at (118.3, 125.3)
- added C91: 22µF, Capacitor_SMD:C_1210_3225Metric, F.Cu at (142.3, 144.6)
- added C92: 22µF, Capacitor_SMD:C_1210_3225Metric, F.Cu at (124.4, 128.9)
- added D3: ON, LED_SMD:LED_0805_2012Metric, F.Cu at (123.0, 86.1)
- added D8: SBRD10200TR, Package_TO_SOT_SMD:ATPAK-2, F.Cu at (104.7, 170.8)
- added D9: B360A-13-F, Libraries:DIOM5226X240N, F.Cu at (89.5, 151.3)
- added IC7: MPQ4423HGQ-P, Libraries:SON65P300X300X100-8N-D, F.Cu at (99.1, 153.5)
- added J5: Conn_01x06, Connector_Molex:Molex_PicoBlade_53047-0610_1x06_P1.25mm_Vertical, F.Cu at (116.9, 93.8)
- added JP1: SolderJumper_3_Open, Jumper:SolderJumper-3_P1.3mm_Open_RoundedPad1.0x1.5mm_NumberLabels, F.Cu at (130.5, 124.1)
- added L2: 10µH 5A, Inductor_SMD:L_12x12mm_H6mm, F.Cu at (92.2, 165.1)
- added L4: 10µH 5A, Inductor_SMD:L_12x12mm_H6mm, F.Cu at (111.5, 153.9)
- added L6: Bead 3A, Inductor_SMD:L_1210_3225Metric, F.Cu at (140.9, 148.5)
- added L7: Bead 3A, Inductor_SMD:L_1210_3225Metric, F.Cu at (119.7, 128.9)
- added M1: Header for 12VDC Fan, Connector_Molex:Molex_KK-254_AE-6410-02A_1x02_P2.54mm_Vertical, F.Cu at (97.6, 132.5)
- added Q3: 2N7002, Package_TO_SOT_SMD:SOT-23, F.Cu at (163.5, 155.4)
- added R11: 1K, Resistor_SMD:R_0603_1608Metric, F.Cu at (251.0, 91.1)
- added R12: 1K, Resistor_SMD:R_0603_1608Metric, F.Cu at (251.0, 94.3)
- added R13: 10kΩ, Resistor_SMD:R_0603_1608Metric, F.Cu at (111.5, 90.6)
- added R14: 10kΩ, Resistor_SMD:R_0603_1608Metric, F.Cu at (116.9, 90.6)
- added R37: 91K, Resistor_SMD:R_0603_1608Metric, F.Cu at (150.7, 147.4)
- added R39: 51K, Resistor_SMD:R_0603_1608Metric, F.Cu at (162.7, 158.0)
- added R42: 10K, Resistor_SMD:R_0603_1608Metric, F.Cu at (159.1, 154.8)
- added R43: 0R, Resistor_SMD:R_0603_1608Metric, F.Cu at (160.6, 154.8)
- added R45: 20K, Resistor_SMD:R_0603_1608Metric, F.Cu at (159.6, 158.0)
- added R47: 10K, Resistor_SMD:R_0603_1608Metric, F.Cu at (144.6, 157.2)
- added R48: 10K, Resistor_SMD:R_0603_1608Metric, B.Cu at (148.0, 151.6)
- added R49: 0.2R, Resistor_SMD:RES_ERJB1CFR036U, F.Cu at (154.8, 162.2)
- added R50: 0.2R, Resistor_SMD:RES_ERJB1CFR036U, F.Cu at (142.7, 160.1)
- added R52: 1M, Resistor_SMD:R_0603_1608Metric, F.Cu at (95.8, 156.2)
- added R55: 2K, Resistor_SMD:R_0603_1608Metric, F.Cu at (84.3, 175.4)
- added R58: 10K, Resistor_SMD:R_0603_1608Metric, F.Cu at (87.7, 177.0)
- added U10: MCP41010T-I/SN, Package_SO:SOIC-8-1EP_3.9x4.9mm_P1.27mm_EP2.29x3mm, F.Cu at (152.6, 141.7)
- added U14: STSPIN820, Libraries:QFN_SPIN820_STM, F.Cu at (148.8, 160.2)
- added U18: TPS55340RTER-TPS55340RTER, Libraries:QFN50P300X300X100-17N, F.Cu at (90.9, 174.3)
- added U19: LM2575-12WU-TR, Package_TO_SOT_SMD:TO-263-5_TabPin3, F.Cu at (88.3, 132.8)
- added U21: LM1117MPX-1.8/NOPB, Package_TO_SOT_SMD:SOT-223-3_TabPin2, F.Cu at (112.6, 128.9)
- added U7: EPM570T100C4N, Package_QFP:LQFP-100_14x14mm_P0.5mm, F.Cu at (130.0, 100.3)
- added U8: STM32F767ZGT6, Package_QFP:LQFP-144_20x20mm_P0.5mm, F.Cu at (161.9, 106.9)
- added X1: Oscillator, Oscillator:Oscillator_SMD_EuroQuartz_XO32-4Pin_3.2x2.5mm, F.Cu at (117.2, 98.7)
- C23: renamed from C30; moved to B.Cu
- C25: renamed from C33; moved to B.Cu
- C41: renamed from C15; moved to B.Cu
- C45: renamed from C90; moved to B.Cu
- D2: renamed from D1; footprint AOD:SOT190P230X110-4N -> Libraries:SOT190P230X110-4N
- J3: value Conn_01x04_Male -> Conn_01x02_Male; footprint Connector_PinHeader_2.54mm:PinHeader_1x04_P2.54mm_Vertical -> Connector_Molex:Molex_KK-254_AE-6410-02A_1x02_P2.54mm_Vertical
- L1: moved to B.Cu
- L3: renamed from L2; value 4.7µH 6.5A -> 220µH 1A; footprint Inductor_SMD:L_Vishay_IHLP-2525 -> Inductor_SMD:L_Wuerth_HCM-7070
- L5: value 10µH 7.2A -> Bead 3A; footprint Inductor_SMD:L_Wuerth_HCI-1050 -> Inductor_SMD:L_1210_3225Metric
- R15: value 10K -> 10kΩ
- R16: value 1K -> 10kΩ
- R17: value 1K -> 330R
- R26: renamed from R14; moved to B.Cu
- R53: value 68.1K -> 64.9 k
- R54: renamed from R59; value 133K -> 20R; footprint Resistor_SMD:R_0402_1005Metric -> Resistor_SMD:R_0603_1608Metric
- R56: value 100kΩ -> 51K; footprint Resistor_SMD:R_0402_1005Metric -> Resistor_SMD:R_0603_1608Metric
- R57: value 9.09K -> 187K; footprint Resistor_SMD:R_0402_1005Metric -> Resistor_SMD:R_0603_1608Metric
- R59: renamed from R63; value 52.3K -> 41.2K
- R60: renamed from R64; value 10K -> 7.68K
- U15: renamed from U20; value DRV8825_STEPPER_MOTOR_DRIVER_CARRIER -> STSPIN820 Stepper Motor Driver Carrier; footprint AOD:DRV8825_STEPPER_MOTOR_DRIVER_CARRIER -> Libraries:SPSPIN820_STEPPER_MOTOR_DRIVER_CARRIER
- U20: renamed from U2; value LM1117-3.3 -> AP2114H-3.3TRG1
- U6: value TPS55340RTER -> MCP4725A0T-E/CH; footprint Libraries:QFN50P300X300X80-17N -> Package_TO_SOT_SMD:SOT-23-6
- U9: renamed from U14; footprint AOD:DRV8825_STEPPER_MOTOR_DRIVER_CARRIER -> Libraries:DRV8825_STEPPER_MOTOR_DRIVER_CARRIER
- moved U6 179.6 mm to (254.6, 92.2), turned to -90 degrees
- moved R15 172.8 mm to (113.1, 90.6), turned to 90 degrees
- moved C55 119.7 mm to (58.7, 106.1), turned to 0 degrees
- moved J3 108.1 mm to (274.4, 92.9), turned to 90 degrees
- moved C83 100.7 mm to (58.8, 82.9), turned to 0 degrees
- moved G2 97.9 mm to (144.9, 64.6)
- moved G1 97.9 mm to (118.3, 65.9)
- moved C64 73.3 mm to (255.0, 131.3), turned to 180 degrees
- moved R16 64.8 mm to (114.6, 90.6), turned to 90 degrees
- moved R17 61.5 mm to (124.0, 89.1), turned to -90 degrees
- moved L1 60.0 mm to (155.4, 94.0)
- moved D6 55.8 mm to (79.0, 78.1)
- moved R28 55.8 mm to (75.6, 78.1)
- moved D5 55.8 mm to (78.9, 74.8)
- moved R27 55.8 mm to (75.6, 74.8)
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- renumbered C71 to C1, C28 to C10, C31 to C11, C35 to C12, C75 to C2, C29 to C22, C32 to C24, C39 to C26, C41 to C27, C43 to C28, C76 to C3, C4 to C32, C5 to C33, C6 to C34, C7 to C35, C9 to C36, C10 to C37, C12 to C38, C13 to C39, C1 to C4, C14 to C40, C16 to C42, C17 to C43, C18 to C44, C88 to C46, C89 to C47, C27 to C48, C79 to C49, C2 to C5, C80 to C50, C81 to C51, C19 to C54, C65 to C55, C85 to C56, C86 to C57, C23 to C58, C25 to C6, C22 to C60, C20 to C62, C21 to C63, C66 to C64, C82 to C65, C83 to C66, C63 to C67, C64 to C68, C67 to C69, C26 to C7, C34 to C70, C36 to C71, C37 to C72, C38 to C73, C68 to C74, C45 to C79, C49 to C80, C74 to C83, C52 to C84, C53 to C86, C8 to C87, C11 to C89, D7 to D1, D5 to D10, D8 to D11, D2 to D4, D4 to D5, D3 to D6, D6 to D7, F2 to F1, F1 to F2, FL2 to FL1, G*** to G1, G*** to G2, H7 to H1, H8 to H2, H9 to H3, H10 to H4, H11 to H5, H12 to H6, IC5 to IC1, IC6 to IC2, IC1 to IC3, IC2 to IC4, IC3 to IC5, IC4 to IC6, J5 to J1, J7 to J10, J13 to J2, J6 to J4, J2 to J6, J1 to J7, MZ2 to MZ1, MZ1 to MZ2, R24 to R1, R5 to R10, R6 to R18, R7 to R19, R25 to R2, R8 to R20, R9 to R21, R10 to R22, R11 to R23, R12 to R24, R13 to R25, R19 to R27, R18 to R28, R31 to R29, R26 to R3, R33 to R30, R34 to R31, R38 to R32, R30 to R33, R67 to R34, R68 to R35, R69 to R36, R32 to R38, R42 to R4, R39 to R40, R37 to R41, R28 to R44, R27 to R46, R20 to R5, R52 to R51, R3 to R6, R54 to R61, R65 to R62, R45 to R7, R49 to R8, R4 to R9, U10 to U1, U19 to U11, U7 to U12, U5 to U13, U24 to U17, U21 to U2, U4 to U3, U8 to U4, U13 to U5
Connections:
- C40 pad 1: +3.3VA -> GND
- C40 pad 2: GND -> +3.3VA
- C41 pad 1: +3.3VA -> GND
- C41 pad 2: GND -> +3.3VA
- C58 pad 1: R-Limit -> Z-Limit
- C79 pad 1: Net-(C45-Pad1) -> Net-(C79-Pad1)
- C89 pad 2: +3V3 -> Net-(C89-Pad2)
- D5 pad 1: /MCU/FSMC_A10 -> /MCU/RED
- D6 pad 1: /MCU/FSMC_A11 -> /MCU/GRN
- IC1 pad 3: Net-(IC5-Pad3) -> unconnected-(IC1-Pad3)
- IC1 pad 4: Net-(IC5-Pad4) -> unconnected-(IC1-Pad4)
- IC2 pad 1: Net-(IC6-Pad1) -> unconnected-(IC2-Pad1)
- IC2 pad 2: Net-(IC6-Pad2) -> unconnected-(IC2-Pad2)
- IC3 pad 1: Net-(IC1-Pad1) -> unconnected-(IC3-Pad1)
- IC3 pad 2: Net-(IC1-Pad2) -> unconnected-(IC3-Pad2)
- IC4 pad 1: Net-(IC2-Pad1) -> unconnected-(IC4-Pad1)
- IC4 pad 2: Net-(IC2-Pad2) -> unconnected-(IC4-Pad2)
- IC5 pad 3: Net-(IC3-Pad3) -> unconnected-(IC5-Pad3)
- IC5 pad 4: Net-(IC3-Pad4) -> unconnected-(IC5-Pad4)
- IC6 pad 1: Net-(IC4-Pad1) -> unconnected-(IC6-Pad1)
- IC6 pad 2: Net-(IC4-Pad2) -> unconnected-(IC6-Pad2)
- J3 pad 1: +5V -> GND
- J3 pad 2: GND -> Net-(C9-Pad1)
- J4 pad 1: Net-(J6-Pad1) -> unconnected-(J4-Pad1)
- J4 pad 4: Net-(J6-Pad4) -> unconnected-(J4-Pad4)
- J4 pad 6: Net-(J6-Pad6) -> unconnected-(J4-Pad6)
- J4 pad 7: Net-(J6-Pad7) -> unconnected-(J4-Pad7)
- J4 pad 8: Net-(J6-Pad8) -> unconnected-(J4-Pad8)
- J4 pad 9: Net-(J6-Pad9) -> unconnected-(J4-Pad9)
- J8 pad 4: Net-(J8-Pad4) -> unconnected-(J8-Pad4)
- J9 pad 4: Net-(J9-Pad4) -> unconnected-(J9-Pad4)
- L5 pad 1: VIN -> Net-(C82-Pad1)
- L5 pad 2: Net-(D11-Pad1) -> +5V
- MZ2 pad 1: Net-(MZ1-Pad1) (its old number) -> /MOTOR/A2
- MZ2 pad 2: Net-(MZ1-Pad2) (its old number) -> /MOTOR/A1
- MZ2 pad 3: Net-(MZ1-Pad3) (its old number) -> /MOTOR/B1
- MZ2 pad 4: Net-(MZ1-Pad4) (its old number) -> /MOTOR/B2
- R15 pad 1: +3V3 -> /MCU/TDI
- R15 pad 2: Net-(R15-Pad2) -> +3V3
- R16 pad 1: /MCU/MCU_SWDIO -> /MCU/TMS
- R17 pad 1: GND -> Net-(D3-Pad2)
- R17 pad 2: /MCU/MCU_SWCLK -> Net-(R17-Pad2)
- R29 pad 1: REN -> ZEN
- R38 pad 1: ZEN -> REN
- R44 pad 1: R-Limit -> Z-Limit
- R51 pad 1: 12V_EN -> +3V3
- R51 pad 2: GND -> 12V_EN
- R54 pad 2: Net-(C48-Pad1) -> Net-(C79-Pad1)
- R56 pad 1: +12V -> Net-(IC7-Pad1)
- R56 pad 2: Net-(C47-Pad2) -> Net-(R56-Pad2)
- R57 pad 1: Net-(C47-Pad2) -> 24V
- R57 pad 2: GND -> Net-(R57-Pad2)
- R59 pad 1: +5V -> Net-(C82-Pad1)
- R59 pad 2: Net-(R63-Pad2) -> Net-(R56-Pad2)
- R60 pad 1: Net-(R63-Pad2) -> Net-(R56-Pad2)
- U1 pad 1: Net-(U10-Pad1) -> unconnected-(U1-Pad1)
- U1 pad 5: Net-(U10-Pad5) -> unconnected-(U1-Pad5)
- U1 pad 6: Net-(U10-Pad6) -> unconnected-(U1-Pad6)
- U1 pad 7: Net-(U10-Pad7) -> unconnected-(U1-Pad7)
- U1 pad 8: Net-(U10-Pad8) -> unconnected-(U1-Pad8)
- U12 pad 4: R-Limit -> Z-Limit
- U15 pad 1: ZEN -> REN
- U15 pad 10: ZFLT -> +3V3
- U15 pad 11: Net-(MZ1-Pad1) (its old number) -> /MOTOR/A2
- U15 pad 12: Net-(MZ1-Pad2) (its old number) -> /MOTOR/A1
- U15 pad 13: Net-(MZ1-Pad3) (its old number) -> /MOTOR/B1
- U15 pad 14: Net-(MZ1-Pad4) (its old number) -> /MOTOR/B2
- U15 pad 2: ZM0 -> RM0
- U15 pad 3: ZM1 -> RM1
- U15 pad 4: ZM2 -> RM2
- U15 pad 7: ZSTEP -> RSTEP
- U15 pad 8: ZDIR -> RDIR
- U20 pad 2: +3V3 -> Net-(C89-Pad2)
- U5 pad 10: Net-(U13-Pad10) -> unconnected-(U5-Pad10)
- U5 pad 7: Net-(U13-Pad7) -> unconnected-(U5-Pad7)
- U5 pad 8: Net-(U13-Pad8) -> unconnected-(U5-Pad8)
- U5 pad 9: Net-(U13-Pad9) -> unconnected-(U5-Pad9)
- U6 pad 1: Net-(D11-Pad1) -> Net-(C9-Pad1)
- U6 pad 2: VIN -> GND
- U6 pad 3: VIN -> +5V
- U6 pad 4: Net-(C69-Pad1) -> SDA
- U6 pad 5: Net-(U6-Pad5) -> SCL
- U9 pad 1: REN -> ZEN
- U9 pad 10: RFLT -> ZFLT
- U9 pad 7: RSTEP -> ZSTEP
- U9 pad 8: RDIR -> ZDIR
Routing:
- net 24V: track 754.6 -> 579.1 mm, vias 9 -> 10
- net /MCU/WK_UP: track 154.2 -> 0.00 mm, vias 2 -> 0
- net SCL: track 0.00 -> 107.7 mm
- net SDA: track 0.00 -> 104.6 mm
- net /MCU/RED: track 0.00 -> 95.4 mm
- net /MCU/GRN: track 0.00 -> 93.4 mm
- net /MCU/FSMC_A11: track 93.1 -> 0.00 mm, vias 2 -> 0
- net /MCU/FSMC_A10: track 91.9 -> 0.00 mm, vias 2 -> 0
- net YFLT: track 82.4 -> 0.00 mm, vias 2 -> 0
- net Net-(C15-Pad2): track 0.00 -> 71.7 mm, vias 0 -> 5
- net SPI3_MOSI: track 0.00 -> 67.3 mm, vias 0 -> 2
- net SPI3_SCK: track 0.00 -> 66.1 mm, vias 0 -> 2
- net +3.3VA: track 68.4 -> 4.99 mm, vias 3 -> 1
- net Net-(BZ1-Pad1): track 0.00 -> 57.7 mm
- net RFLT: track 57.2 -> 0.00 mm, vias 1 -> 0
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- added copper zone on F.Cu, net /MOTOR/A1
- added copper zone on F.Cu, net /MOTOR/A2
- added copper zone on F.Cu, net /MOTOR/B1
- added copper zone on F.Cu, net /MOTOR/B2
- added copper zone on F.Cu, net Net-(C82-Pad1)
- added copper zone on F.Cu, net Net-(D8-Pad1)
- added copper zone on F.Cu, net Net-(R49-Pad2)
- added copper zone on F.Cu, net Net-(R50-Pad2)
- removed copper zone on F.Cu, net Net-(C45-Pad1)
- removed copper zone on F.Cu, net Net-(D11-Pad1)
Other:
- net class Default removed
- net class RF removed
- net class U17 removed
- board text added: "1.8"
- board text added: "13 Apr 2021 初始版 13 Jun 2022 改良版"
- board text added: "3.3"
- board text added: "EPM570(G&Z) use 1.8V Default 3.3V"
- board text removed: "13 Apr 2021 28 Aug 2021"
